Commit message: fixed tf problem

File: gripper/urdf/scene_description.urdf.xacro (robot description, xacro)
@@ -110,5 +110,6 @@
     safety_k_position="$(arg safety_k_position)"
     >
-    <origin xyz="0.35 0.357 0.858" rpy="0.0 0.0 3.1416" />
+    <!-- <origin xyz="0.35 0.357 0.858" rpy="0.0 0.0 3.1416" /> -->
+    <origin xyz="0.0 0.0 0.0" rpy="0.0 0.0 0.0" />
   </xacro:ur_robot>
   <!-- Describe the relationships between the objects -->
@@ -128,9 +129,9 @@
     <origin xyz = "0.4572 0.91 0.895" rpy="1.5708 0 -1.5708" />
   </joint>
-  <!-- <joint name = "small_table_to_ur_base" type="fixed">
+  <joint name = "small_table_to_ur_base" type="fixed">
     <parent link = "small_table"/>
     <child link = "base_link"/>
     <origin xyz="0.35 0.357 0.858" rpy="0.0 0.0 3.1416" />
-  </joint> -->
+  </joint>
   <joint name="robotiq_coupler_joint" type="fixed">
     <parent link="tool0" />

Commit message: actually fixed tf, entire sequence works roughly

File: gripper/urdf/scene_description.urdf.xacro (robot description, xacro)
@@ -110,6 +110,5 @@
     safety_k_position="$(arg safety_k_position)"
     >
-    <!-- <origin xyz="0.35 0.357 0.858" rpy="0.0 0.0 3.1416" /> -->
-    <origin xyz="0.0 0.0 0.0" rpy="0.0 0.0 0.0" />
+    <origin xyz="0.35 0.357 0.858" rpy="0.0 0.0 3.1416" />
   </xacro:ur_robot>
   <!-- Describe the relationships between the objects -->
@@ -129,9 +128,4 @@
     <origin xyz = "0.4572 0.91 0.895" rpy="1.5708 0 -1.5708" />
   </joint>
-  <joint name = "small_table_to_ur_base" type="fixed">
-    <parent link = "small_table"/>
-    <child link = "base_link"/>
-    <origin xyz="0.35 0.357 0.858" rpy="0.0 0.0 3.1416" />
-  </joint>
   <joint name="robotiq_coupler_joint" type="fixed">
     <parent link="tool0" />
